File: schematics/ESP01-PC-WakeUp/ESP01-PC-WakeUp.kicad_pcb (KiCad board)
At the start: 2 copper layers, 65.4 x 21.6 mm, 18 parts, among them J1 JUSB, J2 JUSB, J3 Pin selector, J4 Power, J5 Out 1, J6 Out 2, Q1 BC337, Q2 2N7000, U1 ESP-01, U2 PS2561

Commit message: fix: added the 'JLCJLCJLCJLC' text.
Other:
- board text added: "JLCJLCJLCJLC"
Changed lines of the file:
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@@
     ) (layer "F.SilkS") (width 0.001058) (fill solid))
   (gr_rect (start 236.22 73.66) (end 170.815 95.25) (layer "Edge.Cuts") (width 0.1) (fill none))
+  (gr_text "JLCJLCJLCJLC" (at 230.505 74.93) (layer "B.SilkS")
+    (effects (font (size 1 1) (thickness 0.15)) (justify mirror))
+  )
   (gr_text "TX  RX" (at 202.692 86.868) (layer "F.SilkS")
     (effects (font (size 0.75 0.75) (thickness 0.12)) (justify left))
