File: schematics/ESP01-PC-WakeUp/ESP01-PC-WakeUp.kicad_sch (KiCad schematic)
At the start: 14 parts

Commit message: feat: shematics and footprints
Parts:
- removed J?: JUSB, Connector_PinHeader_2.54mm:PinHeader_2x05_P2.54mm_Vertical, symbol Connector_Generic:Conn_02x05_Odd_Even
- added J2: Pin selector, Connector_PinHeader_2.54mm:PinHeader_2x04_P2.54mm_Vertical, symbol Connector_Generic:Conn_02x04_Odd_Even
- added J3: Power, Connector_PinHeader_2.54mm:PinHeader_2x04_P2.54mm_Vertical, symbol Connector_Generic:Conn_02x04_Odd_Even
- added J4: JUSB, Connector_PinHeader_2.54mm:PinHeader_2x05_P2.54mm_Vertical, symbol Connector_Generic:Conn_02x05_Odd_Even
- added R2: 10k, Resistor_THT:R_Axial_DIN0207_L6.3mm_D2.5mm_P7.62mm_Horizontal, symbol Device:R
- C1, C2: renamed from C?; footprint Capacitor_THT:CP_Radial_D8.0mm_P3.50mm -> Capacitor_THT:CP_Radial_D4.0mm_P1.50mm
- J5: renamed from J?; value OUT -> Out; footprint (none) -> Connector_PinHeader_2.54mm:PinHeader_1x02_P2.54mm_Horizontal
- R5: renamed from R?; footprint (none) -> Resistor_THT:R_Axial_DIN0207_L6.3mm_D2.5mm_P7.62mm_Horizontal
- U2: renamed from U?; footprint Package_DIP:DIP-4_W7.62mm -> Package_DIP:DIP-4_W10.16mm
- gave numbers to parts that had none: 8
Connections:
- net +3V3: now also J3.3 (Pin_3), J3.4 (Pin_4), R2.1; no longer U1.5 (RST)
- net +5V: now also J3.1 (Pin_1), J3.2 (Pin_2), J4.1 (Pin_1), J4.2 (Pin_2)
- net GND: now also J3.5 (Pin_5), J3.6 (Pin_6), J3.8 (Pin_8), J4.7 (Pin_7), J4.8 (Pin_8)
- net PW: now also J2.2 (Pin_2), J2.4 (Pin_4), J2.6 (Pin_6), J2.8 (Pin_8); no longer R4.2, U1.6 (GPIO0)
- net 2: now reaches R3.2, U1.4 (GPIO2)
- net 2: now also J2.3 (Pin_3)
- net D-: now reaches J1.3 (Pin_3)
- net D-: now also J1.4 (Pin_4), J4.3 (Pin_3), J4.4 (Pin_4)
- net D+: now reaches J1.5 (Pin_5)
- net D+: now also J1.6 (Pin_6), J4.5 (Pin_5), J4.6 (Pin_6)
- net TX: now reaches U1.1 (UTXD)
- net TX: now also J2.5 (Pin_5)
- net RX: now reaches U1.8 (URXD)
- net RX: now also J2.7 (Pin_7)
- new net 0: J2.1 (Pin_1), R4.2, U1.6 (GPIO0)
- new net RST: J3.7 (Pin_7), R2.2, U1.5 (RST)
- no-connect marks 12 -> 4
Other:
- note added: "No Pin"
- note removed: "Fare spinotto USB maschio sopra PCB per attaccare l'eventuale cavo USB. Fare pinheader 2x4 con jumper per selezione ed esposizione dei PIN dell'ESP01."
- moved on the sheet: C1, C2, D1, J1, J5, Q1, Q2, R1, R4, R5, U2

Commit message: fix
Parts:
- removed C1, C2: 10u, Capacitor_THT:CP_Radial_D4.0mm_P1.50mm, symbol Device:CP
- added C1, C2: 10u, Capacitor_THT:CP_Radial_D4.0mm_P1.50mm, symbol Device:C_Polarized
Connections:
- net +3V3: now also C2.1
- net +5V: now also C1.1
- net GND: now also C1.2, C2.2
Changed lines of the file:
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@@
 (kicad_sch (version 20211123) (generator eeschema)
   (paper "A4")
+  (junction (at 162.56 64.77) (diameter 0) (color 0 0 0 0)
+  )
   (junction (at 40.64 96.52) (diameter 0) (color 0 0 0 0)
   )
@@
   )
   (junction (at 110.49 53.975) (diameter 0) (color 0 0 0 0)
+  )
+  (junction (at 149.86 57.15) (diameter 0) (color 0 0 0 0)
   )
   (junction (at 162.56 37.465) (diameter 0) (color 0 0 0 0)
@@
     (pin "1")
   )
+  (symbol (lib_id "power:PWR_FLAG") (at 149.86 57.15 0) (unit 1)
+    (in_bom yes) (on_board yes)
+    (property "Reference" "#FLG0101" (id 0) (at 149.86 55.245 0)
+      (effects (font (size 1.27 1.27)) hide)
+    )
+    (property "Value" "PWR_FLAG" (id 1) (at 149.86 52.7558 0)
+      (effects (font (size 1.27 1.27)) hide)
+    )
+    (property "Footprint" "" (id 2) (at 149.86 57.15 0)
+      (effects (font (size 1.27 1.27)) hide)
+    )
+    (property "Datasheet" "~" (id 3) (at 149.86 57.15 0)
+      (effects (font (size 1.27 1.27)) hide)
+    )
+    (pin "1")
+  )
   (symbol (lib_id "power:+3.3V") (at 149.86 59.69 90) (unit 1)
     (in_bom yes) (on_board yes) (fields_autoplaced)
@@
     )
     (pin "1")
+  )
+  (symbol (lib_id "Device:C_Polarized") (at 78.74 96.52 0) (unit 1)
+    (in_bom yes) (on_board yes) (fields_autoplaced)
+    (property "Reference" "C1" (id 0) (at 82.55 94.3609 0)
+      (effects (font (size 1.27 1.27)) (justify left))
+    )
+    (property "Value" "10u" (id 1) (at 82.55 96.9009 0)
+      (effects (font (size 1.27 1.27)) (justify left))
+    )
+    (property "Footprint" "Capacitor_THT:CP_Radial_D4.0mm_P1.50mm" (id 2) (at 79.7052 100.33 0)
+      (effects (font (size 1.27 1.27)) hide)
+    )
+    (property "Datasheet" "~" (id 3) (at 78.74 96.52 0)
+      (effects (font (size 1.27 1.27)) hide)
+    )
+    (pin "1")
+    (pin "2")
   )
   (symbol (lib_id "Connector_Generic:Conn_02x05_Odd_Even") (at 130.175 97.79 90) (unit 1)
@@
     (pin "3")
   )
+  (symbol (lib_id "power:PWR_FLAG") (at 162.56 64.77 270) (unit 1)
+    (in_bom yes) (on_board yes)
+    (property "Reference" "#FLG0102" (id 0) (at 164.465 64.77 0)
+      (effects (font (size 1.27 1.27)) hide)
+    )
+    (property "Value" "PWR_FLAG" (id 1) (at 166.9542 64.77 0)
+      (effects (font (size 1.27 1.27)) hide)
+    )
+    (property "Footprint" "" (id 2) (at 162.56 64.77 0)
+      (effects (font (size 1.27 1.27)) hide)
+    )
+    (property "Datasheet" "~" (id 3) (at 162.56 64.77 0)
+      (effects (font (size 1.27 1.27)) hide)
+    )
+    (pin "1")
+  )
   (symbol (lib_id "power:+5V") (at 153.035 90.17 0) (unit 1)
     (in_bom yes) (on_board yes)
@@
     (pin "2")
   )
-  (symbol (lib_id "Device:CP") (at 91.44 96.52 0) (unit 1)
-    (in_bom yes) (on_board yes)
-    (property "Reference" "C2" (id 0) (at 94.4372 95.3516 0)
-      (effects (font (size 1.27 1.27)) (justify left))
-    )
-    (property "Value" "10u" (id 1) (at 94.4372 97.663 0)
-      (effects (font (size 1.27 1.27)) (justify left))
-    )
-    (property "Footprint" "Capacitor_THT:CP_Radial_D4.0mm_P1.50mm" (id 2) (at 92.4052 100.33 0)
-      (effects (font (size 1.27 1.27)) hide)
-    )
-    (property "Datasheet" "~" (id 3) (at 91.44 96.52 0)
-      (effects (font (size 1.27 1.27)) hide)
-    )
-    (pin "1")
-    (pin "2")
-  )
   (symbol (lib_id "power:+5V") (at 125.095 90.17 0) (unit 1)
     (in_bom yes) (on_board yes)
@@
     )
     (pin "1")
+  )
+  (symbol (lib_id "Device:C_Polarized") (at 91.44 96.52 0) (unit 1)
+    (in_bom yes) (on_board yes) (fields_autoplaced)
+    (property "Reference" "C2" (id 0) (at 95.25 94.3609 0)
+      (effects (font (size 1.27 1.27)) (justify left))
+    )
+    (property "Value" "10u" (id 1) (at 95.25 96.9009 0)
+      (effects (font (size 1.27 1.27)) (justify left))
+    )
+    (property "Footprint" "Capacitor_THT:CP_Radial_D4.0mm_P1.50mm" (id 2) (at 92.4052 100.33 0)
+      (effects (font (size 1.27 1.27)) hide)
+    )
+    (property "Datasheet" "~" (id 3) (at 91.44 96.52 0)
+      (effects (font (size 1.27 1.27)) hide)
+    )
+    (pin "1")
+    (pin "2")
   )
   (symbol (lib_id "power:GND") (at 100.33 36.83 0) (unit 1)
@@
     (pin "2")
   )
-  (symbol (lib_id "Device:CP") (at 78.74 96.52 0) (unit 1)
-    (in_bom yes) (on_board yes)
-    (property "Reference" "C1" (id 0) (at 81.7372 95.3516 0)
-      (effects (font (size 1.27 1.27)) (justify left))
-    )
-    (property "Value" "10u" (id 1) (at 81.7372 97.663 0)
-      (effects (font (size 1.27 1.27)) (justify left))
-    )
-    (property "Footprint" "Capacitor_THT:CP_Radial_D4.0mm_P1.50mm" (id 2) (at 79.7052 100.33 0)
-      (effects (font (size 1.27 1.27)) hide)
-    )
-    (property "Datasheet" "~" (id 3) (at 78.74 96.52 0)
-      (effects (font (size 1.27 1.27)) hide)
-    )
-    (pin "1")
-    (pin "2")
-  )
   (sheet_instances
     (path "/" (page "1"))
@@
       (reference "#FLG01") (unit 1) (value "PWR_FLAG") (footprint "")
     )
+    (path "/79597dda-e65e-4688-8699-52dfc07757e8"
+      (reference "#FLG0101") (unit 1) (value "PWR_FLAG") (footprint "")
+    )
+    (path "/91abd95d-4bfe-4cc7-8378-0f1bc09cce1e"
+      (reference "#FLG0102") (unit 1) (value "PWR_FLAG") (footprint "")
+    )
     (path "/88273dea-bd8b-47dd-ab7c-45689b1d4322"
       (reference "#PWR01") (unit 1) (value "+5V") (footprint "")
@@
       (reference "#PWR030") (unit 1) (value "GND") (footprint "")
     )
-    (path "/f69b8141-8091-474b-aab4-628edc857cd5"
+    (path "/83b570fd-fb78-4343-a291-527366f163b6"
       (reference "C1") (unit 1) (value "10u") (footprint "Capacitor_THT:CP_Radial_D4.0mm_P1.50mm")
     )
-    (path "/ba531765-525a-440f-99fd-1cd985ce4e02"
+    (path "/bc44d6a1-e089-465c-8871-49e57527bc9a"
       (reference "C2") (unit 1) (value "10u") (footprint "Capacitor_THT:CP_Radial_D4.0mm_P1.50mm")
     )

Commit message: feat: Out 2
Parts:
- added J6: Out 2, Connector_PinHeader_2.54mm:PinHeader_1x02_P2.54mm_Horizontal, symbol Connector:Conn_01x02_Male
- J5: value Out -> Out 1
- renumbered J4 to J2, J2 to J3, J3 to J4
Connections:
- net at J5.1 (Pin_1): now also U2.4, J6.1 (Pin_1); no longer U2.3
- net at J5.2 (Pin_2): now also U2.3, J6.2 (Pin_2); no longer U2.4
Other:
- moved on the sheet: J5
Changed lines of the file:
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@@
   (junction (at 149.86 57.15) (diameter 0) (color 0 0 0 0)
   )
+  (junction (at 213.36 65.405) (diameter 0) (color 0 0 0 0)
+  )
   (junction (at 162.56 37.465) (diameter 0) (color 0 0 0 0)
   )
   (junction (at 107.95 44.45) (diameter 0) (color 0 0 0 0)
+  )
+  (junction (at 214.63 61.595) (diameter 0) (color 0 0 0 0)
   )
   (junction (at 162.56 62.23) (diameter 0) (color 0 0 0 0)
@@
   (no_connect (at 163.195 90.17))
   (no_connect (at 135.255 90.17))
+  (wire (pts (xy 213.36 65.405) (xy 213.36 59.055))
+    (stroke (width 0) (type default) (color 0 0 0 0))
+  )
   (wire (pts (xy 133.985 88.9) (xy 132.715 88.9))
     (stroke (width 0) (type default) (color 0 0 0 0))
@@
     (stroke (width 0) (type default) (color 0 0 0 0))
   )
-  (wire (pts (xy 212.09 62.23) (xy 213.36 62.23))
-    (stroke (width 0) (type default) (color 0 0 0 0))
-  )
   (wire (pts (xy 132.715 104.14) (xy 133.985 104.14))
     (stroke (width 0) (type default) (color 0 0 0 0))
   )
+  (wire (pts (xy 214.63 61.595) (xy 214.63 67.945))
+    (stroke (width 0) (type default) (color 0 0 0 0))
+  )
+  (wire (pts (xy 212.09 61.595) (xy 212.09 60.96))
+    (stroke (width 0) (type default) (color 0 0 0 0))
+  )
   (wire (pts (xy 43.815 45.72) (xy 43.815 46.99))
     (stroke (width 0) (type default) (color 0 0 0 0))
@@
     (stroke (width 0) (type default) (color 0 0 0 0))
   )
+  (wire (pts (xy 214.63 61.595) (xy 212.09 61.595))
+    (stroke (width 0) (type default) (color 0 0 0 0))
+  )
   (wire (pts (xy 43.815 46.99) (xy 43.815 48.26))
     (stroke (width 0) (type default) (color 0 0 0 0))
@@
     (stroke (width 0) (type default) (color 0 0 0 0))
   )
-  (wire (pts (xy 213.36 64.77) (xy 212.09 64.77))
-    (stroke (width 0) (type default) (color 0 0 0 0))
-  )
   (wire (pts (xy 160.655 102.87) (xy 160.655 104.14))
     (stroke (width 0) (type default) (color 0 0 0 0))
@@
     (stroke (width 0) (type default) (color 0 0 0 0))
   )
-  (wire (pts (xy 212.09 60.96) (xy 212.09 62.23))
-    (stroke (width 0) (type default) (color 0 0 0 0))
-  )
   (wire (pts (xy 110.49 46.99) (xy 104.14 46.99))
     (stroke (width 0) (type default) (color 0 0 0 0))
@@
     (stroke (width 0) (type default) (color 0 0 0 0))
   )
+  (wire (pts (xy 213.36 59.055) (xy 215.9 59.055))
+    (stroke (width 0) (type default) (color 0 0 0 0))
+  )
   (wire (pts (xy 100.33 36.83) (xy 104.14 36.83))
     (stroke (width 0) (type default) (color 0 0 0 0))
@@
     (stroke (width 0) (type default) (color 0 0 0 0))
   )
-  (wire (pts (xy 212.09 64.77) (xy 212.09 66.04))
+  (wire (pts (xy 215.9 61.595) (xy 214.63 61.595))
+    (stroke (width 0) (type default) (color 0 0 0 0))
+  )
+  (wire (pts (xy 215.9 65.405) (xy 213.36 65.405))
     (stroke (width 0) (type default) (color 0 0 0 0))
   )
@@
     (stroke (width 0) (type default) (color 0 0 0 0))
   )
+  (wire (pts (xy 212.09 65.405) (xy 212.09 66.04))
+    (stroke (width 0) (type default) (color 0 0 0 0))
+  )
   (wire (pts (xy 110.49 53.975) (xy 110.49 46.99))
     (stroke (width 0) (type default) (color 0 0 0 0))
@@
     (stroke (width 0) (type default) (color 0 0 0 0))
   )
+  (wire (pts (xy 214.63 67.945) (xy 215.9 67.945))
+    (stroke (width 0) (type default) (color 0 0 0 0))
+  )
   (wire (pts (xy 43.815 46.99) (xy 55.88 46.99))
     (stroke (width 0) (type default) (color 0 0 0 0))
@@
   )
   (wire (pts (xy 107.95 44.45) (xy 111.76 44.45))
+    (stroke (width 0) (type default) (color 0 0 0 0))
+  )
+  (wire (pts (xy 213.36 65.405) (xy 212.09 65.405))
     (stroke (width 0) (type default) (color 0 0 0 0))
   )
@@
   (symbol (lib_id "Connector_Generic:Conn_02x05_Odd_Even") (at 158.115 97.79 90) (unit 1)
     (in_bom yes) (on_board yes) (fields_autoplaced)
-    (property "Reference" "J4" (id 0) (at 146.685 96.52 0))
+    (property "Reference" "J2" (id 0) (at 146.685 96.52 0))
     (property "Value" "JUSB" (id 1) (at 149.225 96.52 0))
     (property "Footprint" "Connector_PinHeader_2.54mm:PinHeader_2x05_P2.54mm_Vertical" (id 2) (at 158.115 97.79 0)
@@
   (symbol (lib_id "Connector_Generic:Conn_02x04_Odd_Even") (at 154.94 59.69 0) (unit 1)
     (in_bom yes) (on_board yes) (fields_autoplaced)
-    (property "Reference" "J3" (id 0) (at 156.21 50.165 0))
+    (property "Reference" "J4" (id 0) (at 156.21 50.165 0))
     (property "Value" "Power" (id 1) (at 156.21 52.705 0))
     (property "Footprint" "Connector_PinHeader_2.54mm:PinHeader_2x04_P2.54mm_Vertical" (id 2) (at 154.94 59.69 0)
@@
     (pin "2")
   )
+  (symbol (lib_id "Connector:Conn_01x02_Male") (at 220.98 67.945 180) (unit 1)
+    (in_bom yes) (on_board yes) (fields_autoplaced)
+    (property "Reference" "J6" (id 0) (at 222.25 65.4049 0)
+      (effects (font (size 1.27 1.27)) (justify right))
+    )
+    (property "Value" "Out 2" (id 1) (at 222.25 67.9449 0)
+      (effects (font (size 1.27 1.27)) (justify right))
+    )
+    (property "Footprint" "Connector_PinHeader_2.54mm:PinHeader_1x02_P2.54mm_Horizontal" (id 2) (at 220.98 67.945 0)
+      (effects (font (size 1.27 1.27)) hide)
+    )
+    (property "Datasheet" "~" (id 3) (at 220.98 67.945 0)
+      (effects (font (size 1.27 1.27)) hide)
+    )
+    (pin "1")
+    (pin "2")
+  )
   (symbol (lib_id "power:+5V") (at 125.095 90.17 0) (unit 1)
     (in_bom yes) (on_board yes)
@@
     (pin "1")
   )
-  (symbol (lib_id "Connector:Conn_01x02_Male") (at 218.44 64.77 180) (unit 1)
-    (in_bom yes) (on_board yes) (fields_autoplaced)
-    (property "Reference" "J5" (id 0) (at 219.71 62.2299 0)
+  (symbol (lib_id "Connector:Conn_01x02_Male") (at 220.98 61.595 180) (unit 1)
+    (in_bom yes) (on_board yes) (fields_autoplaced)
+    (property "Reference" "J5" (id 0) (at 222.25 59.0549 0)
       (effects (font (size 1.27 1.27)) (justify right))
     )
-    (property "Value" "Out" (id 1) (at 219.71 64.7699 0)
+    (property "Value" "Out 1" (id 1) (at 222.25 61.5949 0)
       (effects (font (size 1.27 1.27)) (justify right))
     )
-    (property "Footprint" "Connector_PinHeader_2.54mm:PinHeader_1x02_P2.54mm_Horizontal" (id 2) (at 218.44 64.77 0)
-      (effects (font (size 1.27 1.27)) hide)
-    )
-    (property "Datasheet" "~" (id 3) (at 218.44 64.77 0)
+    (property "Footprint" "Connector_PinHeader_2.54mm:PinHeader_1x02_P2.54mm_Horizontal" (id 2) (at 220.98 61.595 0)
+      (effects (font (size 1.27 1.27)) hide)
+    )
+    (property "Datasheet" "~" (id 3) (at 220.98 61.595 0)
       (effects (font (size 1.27 1.27)) hide)
     )
@@
   (symbol (lib_id "Connector_Generic:Conn_02x04_Odd_Even") (at 154.94 40.005 0) (unit 1)
     (in_bom yes) (on_board yes) (fields_autoplaced)
-    (property "Reference" "J2" (id 0) (at 156.21 31.115 0))
+    (property "Reference" "J3" (id 0) (at 156.21 31.115 0))
     (property "Value" "Pin selector" (id 1) (at 156.21 33.655 0))
     (property "Footprint" "Connector_PinHeader_2.54mm:PinHeader_2x04_P2.54mm_Vertical" (id 2) (at 154.94 40.005 0)
@@
       (reference "J1") (unit 1) (value "JUSB") (footprint "Connector_PinHeader_2.54mm:PinHeader_2x05_P2.54mm_Vertical")
     )
+    (path "/2d785e51-14ce-497b-b4ad-dd851b18cf59"
+      (reference "J2") (unit 1) (value "JUSB") (footprint "Connector_PinHeader_2.54mm:PinHeader_2x05_P2.54mm_Vertical")
+    )
     (path "/e388fa75-06aa-494e-b294-d4d94b925a4c"
-      (reference "J2") (unit 1) (value "Pin selector") (footprint "Connector_PinHeader_2.54mm:PinHeader_2x04_P2.54mm_Vertical")
+      (reference "J3") (unit 1) (value "Pin selector") (footprint "Connector_PinHeader_2.54mm:PinHeader_2x04_P2.54mm_Vertical")
     )
     (path "/659f63a2-1976-460f-9827-4c547f6cfcd0"
-      (reference "J3") (unit 1) (value "Power") (footprint "Connector_PinHeader_2.54mm:PinHeader_2x04_P2.54mm_Vertical")
-    )
-    (path "/2d785e51-14ce-497b-b4ad-dd851b18cf59"
-      (reference "J4") (unit 1) (value "JUSB") (footprint "Connector_PinHeader_2.54mm:PinHeader_2x05_P2.54mm_Vertical")
+      (reference "J4") (unit 1) (value "Power") (footprint "Connector_PinHeader_2.54mm:PinHeader_2x04_P2.54mm_Vertical")
     )
     (path "/bda55607-6909-4c24-a6e5-a10a75e9ba53"
-      (reference "J5") (unit 1) (value "Out") (footprint "Connector_PinHeader_2.54mm:PinHeader_1x02_P2.54mm_Horizontal")
+      (reference "J5") (unit 1) (value "Out 1") (footprint "Connector_PinHeader_2.54mm:PinHeader_1x02_P2.54mm_Horizontal")
+    )
+    (path "/b7ab2bac-1dd7-46f3-a420-8ab804b7dfe7"
+      (reference "J6") (unit 1) (value "Out 2") (footprint "Connector_PinHeader_2.54mm:PinHeader_1x02_P2.54mm_Horizontal")
     )
     (path "/8dd427e9-0bf4-428e-a522-947f1dc402ae"

Commit message: chore: tidying PCB.
Parts:
- J5, J6: footprint Connector_PinHeader_2.54mm:PinHeader_1x02_P2.54mm_Horizontal -> Connector_PinHeader_2.54mm:PinHeader_1x02_P2.54mm_Vertical
- U2: footprint Package_DIP:DIP-4_W10.16mm -> Package_DIP:DIP-4_W7.62mm
Connections:
- net +5V: now also J1.10 (Pin_10), J1.9 (Pin_9), J2.10 (Pin_10), J2.9 (Pin_9); no longer J1.1 (Pin_1), J1.2 (Pin_2), J2.1 (Pin_1), J2.2 (Pin_2)
- net D-: now also J1.7 (Pin_7), J1.8 (Pin_8), J2.7 (Pin_7), J2.8 (Pin_8); no longer J1.3 (Pin_3), J1.4 (Pin_4), J2.3 (Pin_3), J2.4 (Pin_4)
- net GND: now also J1.3 (Pin_3), J1.4 (Pin_4), J2.3 (Pin_3), J2.4 (Pin_4); no longer J1.7 (Pin_7), J1.8 (Pin_8), J2.7 (Pin_7), J2.8 (Pin_8)
Other:
- moved on the sheet: J1, J2
Changed lines of the file:
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@@
     (pin "1")
   )
-  (symbol (lib_id "Connector_Generic:Conn_02x05_Odd_Even") (at 158.115 97.79 90) (unit 1)
-    (in_bom yes) (on_board yes) (fields_autoplaced)
-    (property "Reference" "J2" (id 0) (at 146.685 96.52 0))
-    (property "Value" "JUSB" (id 1) (at 149.225 96.52 0))
+  (symbol (lib_id "Connector_Generic:Conn_02x05_Odd_Even") (at 158.115 97.79 270) (mirror x) (unit 1)
+    (in_bom yes) (on_board yes) (fields_autoplaced)
+    (property "Reference" "J2" (id 0) (at 169.545 96.52 0))
+    (property "Value" "JUSB" (id 1) (at 167.005 96.52 0))
     (property "Footprint" "Connector_PinHeader_2.54mm:PinHeader_2x05_P2.54mm_Vertical" (id 2) (at 158.115 97.79 0)
       (effects (font (size 1.27 1.27)) hide)
@@
     (pin "2")
   )
-  (symbol (lib_id "Connector_Generic:Conn_02x05_Odd_Even") (at 130.175 97.79 90) (unit 1)
-    (in_bom yes) (on_board yes) (fields_autoplaced)
-    (property "Reference" "J1" (id 0) (at 118.745 96.52 0))
-    (property "Value" "JUSB" (id 1) (at 121.285 96.52 0))
+  (symbol (lib_id "Connector_Generic:Conn_02x05_Odd_Even") (at 130.175 97.79 270) (mirror x) (unit 1)
+    (in_bom yes) (on_board yes) (fields_autoplaced)
+    (property "Reference" "J1" (id 0) (at 141.605 96.52 0))
+    (property "Value" "JUSB" (id 1) (at 139.065 96.52 0))
     (property "Footprint" "Connector_PinHeader_2.54mm:PinHeader_2x05_P2.54mm_Vertical" (id 2) (at 130.175 97.79 0)
       (effects (font (size 1.27 1.27)) hide)
@@
       (effects (font (size 1.27 1.27)) (justify right))
     )
-    (property "Footprint" "Connector_PinHeader_2.54mm:PinHeader_1x02_P2.54mm_Horizontal" (id 2) (at 220.98 67.945 0)
+    (property "Footprint" "Connector_PinHeader_2.54mm:PinHeader_1x02_P2.54mm_Vertical" (id 2) (at 220.98 67.945 0)
       (effects (font (size 1.27 1.27)) hide)
     )
@@
       (effects (font (size 1.27 1.27)) (justify right))
     )
-    (property "Footprint" "Connector_PinHeader_2.54mm:PinHeader_1x02_P2.54mm_Horizontal" (id 2) (at 220.98 61.595 0)
+    (property "Footprint" "Connector_PinHeader_2.54mm:PinHeader_1x02_P2.54mm_Vertical" (id 2) (at 220.98 61.595 0)
       (effects (font (size 1.27 1.27)) hide)
     )
@@
     (property "Reference" "U2" (id 0) (at 204.47 54.61 0))
     (property "Value" "PS2561" (id 1) (at 204.47 57.15 0))
-    (property "Footprint" "Package_DIP:DIP-4_W10.16mm" (id 2) (at 199.39 68.58 0)
+    (property "Footprint" "Package_DIP:DIP-4_W7.62mm" (id 2) (at 199.39 68.58 0)
       (effects (font (size 1.27 1.27) italic) (justify left) hide)
     )
@@
     )
     (path "/bda55607-6909-4c24-a6e5-a10a75e9ba53"
-      (reference "J5") (unit 1) (value "Out 1") (footprint "Connector_PinHeader_2.54mm:PinHeader_1x02_P2.54mm_Horizontal")
+      (reference "J5") (unit 1) (value "Out 1") (footprint "Connector_PinHeader_2.54mm:PinHeader_1x02_P2.54mm_Vertical")
     )
     (path "/b7ab2bac-1dd7-46f3-a420-8ab804b7dfe7"
-      (reference "J6") (unit 1) (value "Out 2") (footprint "Connector_PinHeader_2.54mm:PinHeader_1x02_P2.54mm_Horizontal")
+      (reference "J6") (unit 1) (value "Out 2") (footprint "Connector_PinHeader_2.54mm:PinHeader_1x02_P2.54mm_Vertical")
     )
     (path "/8dd427e9-0bf4-428e-a522-947f1dc402ae"
@@
     )
     (path "/e57aaa28-17df-42b9-8a6c-0a550fb1caf9"
-      (reference "U2") (unit 1) (value "PS2561") (footprint "Package_DIP:DIP-4_W10.16mm")
-    )
-  )
+      (reference "U2") (unit 1) (value "PS2561") (footprint "Package_DIP:DIP-4_W7.62mm")
+    )
+  )
